File: pi5.kicad_pcb (KiCad board)
At the start: 2 copper layers, 310 parts, among them J1 USB_C_Receptacle_GCT_USB4105-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, J10 RJ45_Wuerth_7499111446_Horizo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, J11 USB_A_Wuerth_61400826021_Hori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, J12 USB3_A_Molex_48406-0001_Horiz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, J13 HDMI_Micro-D_Molex_46765-1xxx, J14 PinHeader_2x02_P2.54mm_Vertic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, J17 JST_SH_BM04B-SRSS-TB_1x04-1MP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, J2 HDMI_Micro-D_Molex_46765-1xxx, J20 52559-1652, J3 F32Q-1A7H1-11022, J4 F32Q-1A7H1-11022, J8 PinHeader_2x20_P2.54mm_Vertic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, J9 104031-0811, U5 DA9091

Commit message: new resistor identified
Parts:
- added REF**: 1, Resistor_SMD:R_0201_0603Metric, B.Cu at (158.5, 80.0)
- added REF**: R_0201_0603Metric, Resistor_SMD:R_0201_0603Metric, F.Cu at (158.7, 79.8)
